File: schematics/SCSIknife.kicad_sch (KiCad schematic)
At the start: 91 parts, among them J8 ICSP, K3 LED ACT, K4 USB-C 14-pin, K5 MicroSD Card, K6 SD Card, K8 SD Card extender, U1 RP2040, U10 SN74LVT245, U2 RT5796A, U3 SN74LVT245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

Commit message: Correction to schematics
Parts:
- renumbered C2 to C1, C1 to C2
Changed lines of the file:
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@@
 		(on_board yes)
 		(dnp no)
-		(property "Reference" "C1"
+		(property "Reference" "C2"
 			(at 116.078 37.084 0)
 			(effects
@@
 			(project "SCSIknife"
 				(path "/59c74cdb-6a9b-4f70-b31d-e181008835c9"
-					(reference "C1")
+					(reference "C2")
 					(unit 1)
 				)
@@
 		(on_board yes)
 		(dnp no)
-		(property "Reference" "C2"
+		(property "Reference" "C1"
 			(at 83.058 37.084 0)
 			(effects
@@
 			(project "SCSIknife"
 				(path "/59c74cdb-6a9b-4f70-b31d-e181008835c9"
-					(reference "C2")
+					(reference "C1")
 					(unit 1)
 				)
